File: hardware/piezopiano.sch (EAGLE design)
At the start: 102 parts, among them J1 CON2, Q1 DMN3404L, Q2 DMN3404L, Q3 DMN3404L, Q4 DMN3404L, Q5 DMN3404L, Q6 DMN3404L, Q7 DMN3404L, Q8 DMN3404L, Q9 DNP, U1 ATMEGA4809, U2 CH340E_MSOP10, U5 MSP432P401RIZXHR

Commit message: Wizard speaks
Connections:
- removed net N$1: D11.DIN
- removed net N$21: Q1.G
- net D10~: now also Q1.G
- net D5~: now also D11.DIN
Changed lines of the file:
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@@
 <label x="68.58" y="212.09" size="1.27" layer="95" rot="R180" xref="yes"/>
+</segment>
+<segment>
+<pinref part="D11" gate="G$1" pin="DIN"/>
+<wire x1="195.58" y1="218.44" x2="198.12" y2="218.44" width="0.1524" layer="91"/>
+<label x="198.12" y="218.44" size="1.27" layer="95" xref="yes"/>
 </segment>
 </net>
@@
 <wire x1="73.66" y1="214.63" x2="68.58" y2="214.63" width="0.1524" layer="91"/>
 <label x="68.58" y="214.63" size="1.27" layer="95" rot="R180" xref="yes"/>
+</segment>
+<segment>
+<pinref part="Q1" gate="G$1" pin="G"/>
+<wire x1="233.68" y1="83.82" x2="228.6" y2="83.82" width="0.1524" layer="91"/>
+<label x="228.6" y="83.82" size="1.27" layer="95" rot="R180" xref="yes"/>
 </segment>
 </net>
@@
 </segment>
 </net>
-<net name="N$21" class="0">
-<segment>
-<pinref part="Q1" gate="G$1" pin="G"/>
-<wire x1="233.68" y1="83.82" x2="228.6" y2="83.82" width="0.1524" layer="91"/>
-<label x="228.6" y="83.82" size="1.27" layer="95" rot="R180" xref="yes"/>
-</segment>
-</net>
 <net name="N$22" class="0">
 <segment>
@@
 </segment>
 </net>
-<net name="N$1" class="0">
-<segment>
-<pinref part="D11" gate="G$1" pin="DIN"/>
-<wire x1="195.58" y1="218.44" x2="198.12" y2="218.44" width="0.1524" layer="91"/>
-<label x="198.12" y="218.44" size="1.27" layer="95" xref="yes"/>
-</segment>
-</net>

Commit message: Routing first draft finished
Connections:
- removed net D3: Q2.G
- removed net D5: Q6.G
- removed net D6: Q7.G
- removed net N$37: R35.1
- removed net N$38: R34.1
- removed net N$39: R36.1
- removed net NOTE2: Q4.G
- removed net NOTE5: Q5.G
- removed net T7: C8.1, S6.P, S6.P@1
- removed net X: Q3.G
- removed net Y: Q8.G
- net A0: no longer C9.1, S7.P, S7.P@1
- net A1: no longer C10.1, S8.P, S8.P@1
- net A6: now also C5.1, S3.P, S3.P@1
- net A7: now also C6.1, S4.P, S4.P@1
- net D2: now also Q8.G; no longer C5.1, S3.P, S3.P@1
- net D3~: now also R35.1
- net D6~: now also R36.1
- net D7: now also Q7.G; no longer C6.1, S4.P, S4.P@1
- net D8: now also C8.1, S6.P, S6.P@1
- net D9~: now also R34.1
- net PA04: now also Q6.G; no longer C7.1, S5.P, S5.P@1
- net PA05: now also Q5.G
- net PA06: now also Q4.G
- net PA07: now also Q3.G
- net PB03: now also Q2.G
- net PD06: now also C7.1, S5.P, S5.P@1
- net PF00: now also C9.1, S7.P, S7.P@1
- net PF01: now also C10.1, S8.P, S8.P@1

Commit message: Renumbered, Gerbers Created
Parts:
- removed R36: 1k, zaan-Resistors:1KOHM-0603-1/10W-1%
- added R33: 1k, zaan-Resistors:1KOHM-0603-1/10W-1%
- C1, C2: value 100n -> 22u; device zaan-Capacitors:100NF-0603-50V-5% -> zaan-Capacitors:22UF-0805-25V-20%
- C14, C15: value 22u -> 100n; device zaan-Capacitors:22UF-0805-25V-20% -> zaan-Capacitors:100NF-0603-50V-5%
- D11: value WS2812B -> LED_YELLOW; device zaan-Optoelectronics:WS2812B -> zaan-Optoelectronics:CHIP-FLAT-Y_0603-0.55MM
- D12: value LED_YELLOW -> (none); device zaan-Optoelectronics:CHIP-FLAT-Y_0603-0.55MM -> zaan-Optoelectronics:150121M173000
- D3: value (none) -> WS2812B; device zaan-Optoelectronics:150121M173000 -> zaan-Optoelectronics:WS2812B
- J1: value CON2 -> (none); device Custom:CON2 -> zaan-Connectors:USB_C2-LAYER
- J2: value (none) -> CON2; device zaan-Connectors:USB_C2-LAYER -> Custom:CON2
- R1, R11, R13, R5, R7, R9: value 10k -> 1k; device zaan-Resistors:10KOHM-0603-1/10W-1% -> zaan-Resistors:1KOHM-0603-1/10W-1%
- R10, R12, R14, R4, R6, R8: value 100R -> 1k; device zaan-Resistors:100OHM-0603-1/10W-1% -> zaan-Resistors:1KOHM-0603-1/10W-1%
- R17, R21, R23, R25, R27, R29: value 1k -> 10k; device zaan-Resistors:1KOHM-0603-1/10W-1% -> zaan-Resistors:10KOHM-0603-1/10W-1%
- R18: value 5.1k -> 100R; device zaan-Resistors:5.1KOHM-0603-1/10W-1% -> zaan-Resistors:100OHM-0603-1/10W-1%
- R19: value 5.1k -> 10k; device zaan-Resistors:5.1KOHM-0603-1/10W-1% -> zaan-Resistors:10KOHM-0603-1/10W-1%
- R2: value 100R -> 5.1k; device zaan-Resistors:100OHM-0603-1/10W-1% -> zaan-Resistors:5.1KOHM-0603-1/10W-1%
- R20, R22, R24, R26, R28, R30: value 1k -> 100R; device zaan-Resistors:1KOHM-0603-1/10W-1% -> zaan-Resistors:100OHM-0603-1/10W-1%
- R3: value 10k -> 5.1k; device zaan-Resistors:10KOHM-0603-1/10W-1% -> zaan-Resistors:5.1KOHM-0603-1/10W-1%
- R31: value DNP -> 1k; device zaan-Resistors:DNP-0603 -> zaan-Resistors:1KOHM-0603-1/10W-1%
- R32: value DNP -> 1k; device zaan-Resistors:DNP-0805 -> zaan-Resistors:1KOHM-0603-1/10W-1%
- R34: value 1k -> DNP; device zaan-Resistors:1KOHM-0603-1/10W-1% -> zaan-Resistors:DNP-0805
- R35: value 1k -> DNP; device zaan-Resistors:1KOHM-0603-1/10W-1% -> zaan-Resistors:DNP-0603
- U1: value ATMEGA4809 -> CH340E_MSOP10; device zaan-IC-Microcontroller:ATMEGA4809 -> zaan-IC-General:CH340E_MSOP10
- U2: value CH340E_MSOP10 -> ATMEGA4809; device zaan-IC-General:CH340E_MSOP10 -> zaan-IC-Microcontroller:ATMEGA4809
- renumbered U5 to U3
Connections:
- net +5V: now also C4.1, C5.1, C6.1, C7.1, D12.4, D3.VDD, J2.2, JP1.1, R1.1, R10.2, R12.2, R14.2, R17.2, R19.2, R21.2, R23.2, R8.2, U1.VCC, U2.AVDD, U2.VDD@1, U2.VDD@2; no longer C12.1, C13.1, C14.1, C15.1, D11.VDD, D3.4, J1.2, JP6.1, R1.2, R17.1, R20.2, R24.2, R26.2, R28.2, R3.2, R30.2, R5.2, U1.AVDD, U1.VDD@1, U1.VDD@2, U2.VCC
- net A0: now also JP6.1, U2.PD03; no longer JP1.1, U1.PD03
- net A1: now also JP5.1, U2.PD02; no longer JP2.1, U1.PD02
- net A2: now also JP4.1, U2.PD01; no longer JP3.1, U1.PD01
- net A3: now also JP3.1, U2.PD00; no longer JP4.1, U1.PD00
- net A4/SDA: now also U2.PA02; no longer U1.PA02
- net A5/SCL: now also U2.PA03; no longer U1.PA03
- net A6: now also C10.1, U2.PD04; no longer C5.1, U1.PD04
- net A7: now also C11.1, U2.PD05; no longer C6.1, U1.PD05
- net AREF: now also U2.PD07; no longer U1.PD07
- net D10~: now also U2.PB01; no longer U1.PB01
- net D2: now also U2.(EXTCLK)PA00; no longer U1.(EXTCLK)PA00
- net D3~: now also R31.1, U2.PF05; no longer R35.1, U1.PF05
- net D4: now also C8.1, U2.PC06; no longer C3.1, U1.PC06
- net D5~: now also D3.DIN, U2.PB02; no longer D11.DIN, U1.PB02
- net D6~: now also R32.1, U2.PF04; no longer R36.1, U1.PF04
- net D7: now also U2.PA01; no longer U1.PA01
- net D8: now also C13.1, U2.PE03; no longer C8.1, U1.PE03
- net D9~: now also R33.1, U2.PB00; no longer R34.1, U1.PB00
- net GND: now also D1.C, D2.C, D3.VSS, J1.GND, J1.SHLD, J2.1, JP2.1, R2.1, R3.1, U1.GND, U2.GND@1, U2.GND@2, U2.GND@3; no longer D11.VSS, D12.C, D4.C, J1.1, J2.GND, J2.SHLD, JP5.1, R18.1, R19.1, U1.GND@1, U1.GND@2, U1.GND@3, U2.GND
- net MISO: now also U2.PE01; no longer U1.PE01
- net MOSI: now also U2.PE00; no longer U1.PE00
- net N$10: now also LS8.2, R21.1, R22.2; no longer LS3.2, R7.1, R8.2
- net N$11: now also LS3.2, R15.1, R16.2; no longer LS5.2, R1.1, R2.2
- net N$12: now also D5.C, R18.1; no longer D10.C, R4.1
- net N$13: now also LS5.2, R23.1, R24.2; no longer LS8.2, R10.2, R9.1
- net N$14: now also D9.C, R26.1; no longer D7.C, R12.1
- net N$15: now also R29.1, R30.2; no longer R15.1, R16.2
- net N$16: now also LS7.2, R27.1, R28.2; no longer LS6.2, R13.1, R14.2
- net N$17: now also D10.C, R28.1; no longer D9.C, R14.1
- net N$18: now also LS1.2, R19.1, R20.2; no longer LS7.2, R5.1, R6.2
- net N$19: now also R5.1, U1.TNOW; no longer R23.1, U2.TNOW
- net N$2: now also D7.C, R22.1; no longer D6.C, R8.1
- net N$20: now also D2.A, R5.2; no longer D4.A, R23.2
- net N$22: now also D6.A, R9.1; no longer D2.A, R24.1
- net N$23: now also D8.A, R11.1; no longer D5.A, R29.1
- net N$24: now also D9.A, R12.1; no longer D7.A, R30.1
- net N$25: now also D7.A, R10.1; no longer D6.A, R20.1
- net N$26: now also D11.A, R14.1; no longer D8.A, R27.1
- net N$27: now also D4.A, R7.1; no longer D1.A, R28.1
- net N$28: now also D12.R, R31.2; no longer D3.R, R35.2
- net N$29: now also J1.CC2, R3.2; no longer J2.CC2, R18.2
- net N$3: now also D4.C, R16.1; no longer D1.C, R2.1
- net N$30: now also J1.CC1, R2.2; no longer J2.CC1, R19.2
- net N$31: now also J1.D+, U1.UD+; no longer J2.D+, U2.UD+
- net N$32: now also J1.D-, U1.UD-; no longer J2.D-, U2.UD-
- net N$33: now also D5.A, R8.1; no longer D10.A, R25.1
- net N$34: now also D10.A, R13.1; no longer D9.A, R26.1
- net N$35: now also D12.G, R33.2; no longer D3.G, R34.2
- net N$36: now also D12.B, R32.2; no longer D3.B, R36.2
- net N$4: now also LS6.2, R17.1, R18.2; no longer LS2.2, R3.1, R4.2
- net N$5: now also D8.C, R24.1; no longer D5.C, R10.1
- net N$6: now also LS2.2, R25.1, R26.2; no longer LS1.2, R11.1, R12.2
- net N$7: now also D11.C, R30.1; no longer D8.C, R16.1
- net N$8: now also D1.A, R1.2; no longer D12.A, R17.2
- net N$9: now also D6.C, R20.1; no longer D2.C, R6.1
- net PA04: now also U2.PA04; no longer U1.PA04
- net PA05: now also U2.PA05; no longer U1.PA05
- net PA06: now also U2.PA06; no longer U1.PA06
- net PA07: now also U2.PA07; no longer U1.PA07
- net PB03: now also U2.PB03; no longer U1.PB03
- net PC00: now also U2.PC00; no longer U1.PC00
- net PC01: now also U2.PC01; no longer U1.PC01
- net PC02: now also U2.PC02; no longer U1.PC02
- net PC03: now also U2.PC03; no longer U1.PC03
- net PC07: now also C9.1, U2.PC07; no longer C4.1, U1.PC07
- net PD06: now also C12.1, U2.PD06; no longer C7.1, U1.PD06
- net PF00: now also C14.1, U2.PF00; no longer C9.1, U1.PF00
- net PF01: now also C15.1, U2.PF01; no longer C10.1, U1.PF01
- net PF02: now also U2.PF02; no longer U1.PF02
- net PF03: now also U2.PF03; no longer U1.PF03
- net RESETN: now also U2.RST/PF06; no longer U1.RST/PF06
- net RX0: now also R4.1, U2.PB05; no longer R21.1, U1.PB05
- net RX1: now also U2.PC05; no longer U1.PC05
- net RXD: now also R6.2, U1.RXD; no longer R22.2, U2.RXD
- net SCK: now also U2.PE02; no longer U1.PE02
- net TX0: now also R6.1, U2.PB04; no longer R22.1, U1.PB04
- net TX1: now also U2.PC04; no longer U1.PC04
- net TXD: now also R4.2, U1.TXD; no longer R21.2, U2.TXD
- net UDPI: now also U2.UPDI; no longer U1.UPDI
- net V3: now also C3.1, U1.V3; no longer C11.1, U2.V3
- net VBUS: now also J1.VBUS; no longer J2.VBUS
Other:
- moved on the sheet: C1, C10, C11, C12, C13, C14, C15, C2, C3, C4, C5, C6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
